Commit message: Minimal description package

File: furbot_description/urdf/furbot.urdf (robot description, URDF)
Before this commit: robot furbot_burger, 4 links, 3 joints
Links:
- link base_link: geometry collision box size=0.2 0.4 0.7; visual box size=0.2 0.4 0.7
- link wheel_left_link: geometry collision cylinder length=0.05 radius=0.2; visual cylinder length=0.05 radius=0.2
- link wheel_right_link: geometry collision cylinder length=0.05 radius=0.2; visual cylinder length=0.05 radius=0.2
Joints:
- joint base_joint: origin xyz=0.0 0.0 0.010 rpy=0 0 0 -> xyz=0.0 0.0 0.20 rpy=0 0 0
- joint wheel_left_joint: origin xyz=0.0 0.08 0.023 rpy=-1.57 0 0 -> xyz=0.0 0.25 0.0 rpy=-1.57 0 0
- joint wheel_right_joint: origin xyz=0.0 -0.080 0.023 rpy=-1.57 0 0 -> xyz=0.0 -0.25 0.0 rpy=1.57 0 0

Commit message: Fix wheel axis

File: furbot_description/urdf/furbot.urdf (robot description, URDF)
Before this commit: robot furbot_burger, 4 links, 3 joints
Joints:
- joint wheel_left_joint: axis 0 0 1 -> 0 1 0
- joint wheel_right_joint: axis 0 0 1 -> 0 1 0

Commit message: Updates after galactic install

File: furbot_description/urdf/furbot.urdf (robot description, URDF)
Before this commit: robot furbot_burger, 4 links, 3 joints
Joints:
- joint wheel_left_joint: origin xyz=0.0 0.25 0.0 rpy=-1.57 0 0 -> xyz=0.0 0.25 0.0 rpy=0 0 0
- joint wheel_right_joint: origin xyz=0.0 -0.25 0.0 rpy=1.57 0 0 -> xyz=0.0 -0.25 0.0 rpy=0 0 0

Commit message: Add IMU sensor in webots simulation

File: furbot_description/urdf/furbot.urdf (robot description, URDF)
Before this commit: robot furbot_burger, 4 links, 3 joints
Links:
- added link imu_link
Joints:
- added joint imu_joint: type fixed, parent base_link, child imu_link, origin xyz=0.0 0.0 0.125 rpy=0 0 0
